File: fami.brd (EAGLE design)
At the start: 91.4 x 50.8 mm, 14 parts, among them IC1 PROM, IC2 WRAM, IC3 CHROM, IC4 74LS20N

Commit message: optimized the pcb a little bit
Parts:
- moved R1 22.9 mm to (44.5, 48.3), turned to 180 degrees
- moved D2 20.8 mm to (35.6, 48.3), turned to 0 degrees
- moved R2 20.5 mm to (44.5, 45.7), turned to 0 degrees
- moved JP1 2.54 mm to (26.7, 25.4)
- moved G2 2.54 mm to (11.4, 38.1)
Routing:
- net N$24: track 73.2 -> 40.2 mm
- net N$4: track 15.3 -> 36.2 mm
- net N$6: track 30.3 -> 34.6 mm
- net VRAMA10: track 45.9 -> 47.7 mm
- net PA11: track 49.7 -> 50.9 mm
- net PA10: track 32.7 -> 33.7 mm
Other:
- board size 91.4 x 50.8 mm -> 86.4 x 50.8 mm
Changed lines of the file:
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@@
 <board>
 <plain>
-<text x="25.4" y="26.67" size="1.778" layer="16" font="vector" ratio="15" rot="MR0">V</text>
-<text x="19.05" y="26.67" size="1.778" layer="16" font="vector" ratio="15" rot="MR0">H</text>
+<text x="29.21" y="24.13" size="1.778" layer="16" font="vector" ratio="15" rot="MR0">V</text>
+<text x="20.32" y="24.13" size="1.778" layer="16" font="vector" ratio="15" rot="MR0">H</text>
 <text x="35.56" y="12.7" size="1.778" layer="16" font="vector" ratio="15" rot="MR0">CHR</text>
 <text x="81.28" y="12.7" size="1.778" layer="16" font="vector" ratio="15" rot="MR0">PRG</text>
 <text x="74.93" y="38.1" size="1.778" layer="16" font="vector" ratio="15" rot="MR0">WRAM</text>
-<wire x1="83.185" y1="0" x2="87.63" y2="0" width="0" layer="20"/>
-<wire x1="0.635" y1="0" x2="-3.81" y2="0" width="0" layer="20"/>
-<wire x1="-3.81" y1="0" x2="-3.81" y2="50.8" width="0" layer="20"/>
-<wire x1="-3.81" y1="50.8" x2="87.63" y2="50.8" width="0" layer="20"/>
-<wire x1="87.63" y1="50.8" x2="87.63" y2="0" width="0" layer="20"/>
+<wire x1="83.185" y1="0" x2="85.09" y2="0" width="0" layer="20"/>
+<wire x1="0.635" y1="0" x2="-1.27" y2="0" width="0" layer="20"/>
+<wire x1="-1.27" y1="0" x2="-1.27" y2="50.8" width="0" layer="20"/>
+<wire x1="-1.27" y1="50.8" x2="85.09" y2="50.8" width="0" layer="20"/>
+<wire x1="85.09" y1="50.8" x2="85.09" y2="0" width="0" layer="20"/>
 </plain>
 <attributes>
@@
 <element name="IC4" library="74xx-eu" package="DIL14" value="74LS20N" x="31.75" y="36.83" rot="MR90"/>
 <element name="D1" library="diode" package="D-5" value="" x="77.47" y="35.56" rot="MR270"/>
-<element name="D2" library="diode" package="D-5" value="" x="22.86" y="31.75" rot="MR270"/>
-<element name="JP1" library="SparkFun-Connectors" package="1X03" value="" x="24.13" y="25.4" rot="MR0"/>
+<element name="D2" library="diode" package="D-5" value="" x="35.56" y="48.26" rot="MR0"/>
+<element name="JP1" library="SparkFun-Connectors" package="1X03" value="" x="26.67" y="25.4" rot="MR0"/>
 <element name="C1" library="rcl" package="E2,5-6" value="" x="78.74" y="43.18"/>
 <element name="C2" library="rcl" package="C025-025X050" value="" x="33.02" y="25.4" rot="R180"/>
-<element name="R1" library="rcl" package="0204/7" value="" x="22.86" y="40.64" rot="R270"/>
-<element name="R2" library="rcl" package="0204/7" value="" x="25.4" y="38.1" rot="R270"/>
+<element name="R1" library="rcl" package="0204/7" value="" x="44.45" y="48.26" rot="R180"/>
+<element name="R2" library="rcl" package="0204/7" value="" x="44.45" y="45.72"/>
 <element name="C3" library="rcl" package="C025-025X050" value="" x="74.93" y="24.13" rot="R90"/>
-<element name="G2" library="battery" package="B2430UNI" value="B2430UNI" x="8.89" y="38.1" rot="R180"/>
+<element name="G2" library="battery" package="B2430UNI" value="B2430UNI" x="11.43" y="38.1" rot="R180"/>
 </elements>
 <signals>
@@
 <contactref element="IC2" pad="26"/>
 <polygon width="0.254" layer="16">
-<vertex x="-2.54" y="49.53"/>
-<vertex x="86.36" y="49.53"/>
-<vertex x="86.36" y="1.27"/>
-<vertex x="-2.54" y="1.27"/>
+<vertex x="0" y="49.53"/>
+<vertex x="83.82" y="49.53"/>
+<vertex x="83.82" y="1.27"/>
+<vertex x="0" y="1.27"/>
 </polygon>
 <wire x1="40.64" y1="-5.715" x2="40.64" y2="2.54" width="0.6096" layer="16"/>
@@
 <wire x1="21.59" y1="7.62" x2="21.59" y2="11.43" width="0.254" layer="1"/>
 <wire x1="21.59" y1="11.43" x2="17.78" y2="15.24" width="0.254" layer="1"/>
-<wire x1="17.78" y1="15.24" x2="17.78" y2="22.86" width="0.254" layer="1"/>
-<wire x1="17.78" y1="22.86" x2="16.51" y2="24.13" width="0.254" layer="1"/>
-<wire x1="16.51" y1="24.13" x2="16.51" y2="26.14395" width="0.254" layer="1"/>
-<wire x1="24.13" y1="20.32" x2="24.13" y2="25.4" width="0.254" layer="1"/>
-<wire x1="16.51" y1="26.14395" x2="18.30605" y2="27.94" width="0.254" layer="1"/>
-<wire x1="18.30605" y1="27.94" x2="22.86" y2="27.94" width="0.254" layer="1"/>
-<wire x1="22.86" y1="27.94" x2="24.13" y2="26.67" width="0.254" layer="1"/>
-<wire x1="24.13" y1="26.67" x2="24.13" y2="25.4" width="0.254" layer="1"/>
+<wire x1="17.78" y1="15.24" x2="17.78" y2="25.10019375" width="0.254" layer="1"/>
+<wire x1="17.78" y1="25.10019375" x2="20.61980625" y2="27.94" width="0.254" layer="1"/>
+<wire x1="20.61980625" y1="27.94" x2="25.4" y2="27.94" width="0.254" layer="1"/>
+<wire x1="24.13" y1="20.32" x2="24.13" y2="22.11605" width="0.254" layer="1"/>
+<wire x1="24.13" y1="22.11605" x2="24.87395" y2="22.86" width="0.254" layer="1"/>
+<wire x1="24.87395" y1="22.86" x2="26.67" y2="24.65605" width="0.254" layer="1"/>
+<wire x1="26.67" y1="24.65605" x2="26.67" y2="25.4" width="0.254" layer="1"/>
+<wire x1="25.4" y1="27.94" x2="26.67" y2="26.67" width="0.254" layer="1"/>
+<wire x1="26.67" y1="26.67" x2="26.67" y2="25.4" width="0.254" layer="1"/>
 </signal>
 <signal name="PA9">
@@
 <wire x1="22.86" y1="12.7" x2="19.05" y2="16.51" width="0.254" layer="1"/>
 <wire x1="19.05" y1="16.51" x2="19.05" y2="20.32" width="0.254" layer="1"/>
-<wire x1="19.05" y1="20.32" x2="19.05" y2="25.4" width="0.254" layer="1"/>
+<wire x1="19.05" y1="20.32" x2="19.05" y2="22.86" width="0.254" layer="1"/>
+<wire x1="19.05" y1="22.86" x2="21.59" y2="25.4" width="0.254" layer="1"/>
 </signal>
 <signal name="RW">
@@
 <wire x1="73.66" y1="43.18" x2="77.47" y2="43.18" width="0.6096" layer="16"/>
 <wire x1="77.47" y1="43.18" x2="77.47" y2="38.1" width="0.6096" layer="16"/>
-<wire x1="72.39" y1="45.72" x2="24.13" y2="45.72" width="0.6096" layer="16"/>
-<wire x1="24.13" y1="45.72" x2="22.86" y2="44.45" width="0.6096" layer="16"/>
-<wire x1="72.39" y1="45.72" x2="73.66" y2="44.45" width="0.6096" layer="16"/>
-<wire x1="73.66" y1="44.45" x2="73.66" y2="43.18" width="0.6096" layer="16"/>
+<wire x1="48.26" y1="48.26" x2="70.82019375" y2="48.26" width="0.6096" layer="16"/>
+<wire x1="70.82019375" y1="48.26" x2="73.66" y2="45.42019375" width="0.6096" layer="16"/>
+<wire x1="73.66" y1="45.42019375" x2="73.66" y2="43.18" width="0.6096" layer="16"/>
 <contactref element="C1" pad="+"/>
 <contactref element="R2" pad="2"/>
 <contactref element="R1" pad="1"/>
-<wire x1="25.4" y1="34.29" x2="25.4" y2="38.1" width="0.254" layer="1"/>
-<wire x1="25.4" y1="38.1" x2="22.86" y2="40.64" width="0.254" layer="1"/>
-<wire x1="22.86" y1="40.64" x2="22.86" y2="44.45" width="0.254" layer="1"/>
+<wire x1="48.26" y1="45.72" x2="48.26" y2="48.26" width="0.254" layer="1"/>
 </signal>
 <signal name="N$6">
 <contactref element="IC2" pad="20"/>
 <contactref element="IC4" pad="6"/>
-<wire x1="31.75" y1="40.64" x2="52.07" y2="40.64" width="0.254" layer="1"/>
+<wire x1="31.75" y1="40.64" x2="38.1" y2="40.64" width="0.254" layer="1"/>
+<wire x1="38.1" y1="40.64" x2="52.07" y2="40.64" width="0.254" layer="1"/>
 <wire x1="52.07" y1="40.64" x2="53.34" y2="41.91" width="0.254" layer="1"/>
 <wire x1="53.34" y1="41.91" x2="53.34" y2="43.18" width="0.254" layer="1"/>
@@
 <wire x1="30.48" y1="41.91" x2="27.94" y2="41.91" width="0.254" layer="1"/>
 <contactref element="R2" pad="1"/>
-<wire x1="27.94" y1="41.91" x2="25.4" y2="41.91" width="0.254" layer="1"/>
+<wire x1="40.64" y1="45.72" x2="39.37" y2="45.72" width="0.254" layer="1"/>
+<wire x1="39.37" y1="45.72" x2="38.1" y2="44.45" width="0.254" layer="1"/>
+<wire x1="38.1" y1="44.45" x2="38.1" y2="40.64" width="0.254" layer="1"/>
 </signal>
 <signal name="O2">
@@
 <wire x1="19.05" y1="8.6251" x2="19.05" y2="16.51" width="0.254" layer="16"/>
 <via x="20.32" y="17.78" extent="1-16" drill="0.6"/>
-<wire x1="20.32" y1="17.78" x2="20.32" y2="22.86" width="0.254" layer="1"/>
-<wire x1="20.32" y1="22.86" x2="21.59" y2="24.13" width="0.254" layer="1"/>
-<wire x1="21.59" y1="24.13" x2="21.59" y2="25.4" width="0.254" layer="1"/>
+<wire x1="20.32" y1="17.78" x2="20.32" y2="21.59" width="0.254" layer="1"/>
+<wire x1="20.32" y1="21.59" x2="21.59" y2="22.86" width="0.254" layer="1"/>
+<wire x1="21.59" y1="22.86" x2="22.86" y2="22.86" width="0.254" layer="1"/>
+<wire x1="22.86" y1="22.86" x2="24.13" y2="24.13" width="0.254" layer="1"/>
+<wire x1="24.13" y1="24.13" x2="24.13" y2="25.4" width="0.254" layer="1"/>
 </signal>
 <signal name="N$1">
 <contactref element="R1" pad="2"/>
 <contactref element="D2" pad="C"/>
-<wire x1="22.86" y1="34.29" x2="22.86" y2="36.83" width="0.6096" layer="16"/>
+<wire x1="38.1" y1="48.26" x2="40.64" y2="48.26" width="0.6096" layer="16"/>
 </signal>
 <signal name="N$4">
 <contactref element="D2" pad="A"/>
 <contactref element="G2" pad="+@4"/>
-<wire x1="22.86" y1="29.21" x2="12.065" y2="29.21" width="0.6096" layer="16"/>
-<wire x1="12.065" y1="29.21" x2="8.89" y2="26.035" width="0.6096" layer="16"/>
+<wire x1="11.43" y1="26.035" x2="11.43" y2="35.18455" width="0.6096" layer="16"/>
+<wire x1="11.43" y1="35.18455" x2="24.50545" y2="48.26" width="0.6096" layer="16"/>
+<wire x1="24.50545" y1="48.26" x2="33.02" y2="48.26" width="0.6096" layer="16"/>
 </signal>
 </signals>
